File: KiCAD/Radar.kicad_pcb (KiCad board)
At the start: 2 copper layers, 15 parts

Commit message: Layout V2
Parts:
- added U3: HB100, Footprinty:HB100, F.Cu at (55.5, 121.5)
- added U4: NUCLEO-L432KC, Footprinty:MODULE_NUCLEO-L432KC, F.Cu at (248.4, 121.7)
- added U5: LM358DR, Footprinty:D8, F.Cu at (173.2, 110.9)
- moved C7 128.9 mm to (20.9, 127.5)
- moved R4 69.0 mm to (92.4, 136.5)
- moved C6 51.4 mm to (196.6, 111.0)
- moved R8 51.4 mm to (205.3, 113.5)
- moved R1 45.8 mm to (105.5, 90.0)
- moved R2 45.8 mm to (105.5, 92.5)
- moved C1 45.8 mm to (101.1, 90.0)
- moved C2 42.8 mm to (106.0, 119.5)
- moved R3 35.9 mm to (122.9, 120.0)
- moved C3 15.0 mm to (140.8, 115.5)
- moved R5 15.0 mm to (155.6, 108.0)
- moved R7 15.0 mm to (155.6, 113.0)
- moved C4 15.0 mm to (146.8, 110.5)
- moved C5 15.0 mm to (140.8, 121.3)
- moved R6 15.0 mm to (155.6, 110.5)
Connections:
- net Net-(C1-Pad1) renamed 2IN+
- net Net-(C2-Pad1) renamed 1IN+
- net Net-(C6-Pad1) renamed 2IN-
- net Net-(U4B-PA3) renamed 2OUT

Commit message: PCB V1
Parts:
- moved C7 114.5 mm to (130.0, 92.9), turned to -90 degrees
- moved U3 107.9 mm to (149.5, 68.5), turned to 90 degrees
- moved U4 96.4 mm to (152.1, 127.1), turned to 90 degrees
- moved R4 60.1 mm to (138.5, 98.0), turned to -90 degrees
- moved R8 52.8 mm to (152.6, 112.1), turned to 90 degrees
- moved C6 46.6 mm to (150.1, 112.1), turned to 90 degrees
- moved C1 35.7 mm to (129.7, 111.4), turned to -90 degrees
- moved R1 35.7 mm to (134.1, 111.4), turned to -90 degrees
- moved C2 34.3 mm to (133.6, 99.2), turned to 90 degrees
- moved R2 29.9 mm to (131.6, 107.1)
- moved C5 28.3 mm to (166.1, 108.6), turned to 90 degrees
- moved U5 27.4 mm to (146.1, 106.6), turned to -90 degrees
- moved R3 18.9 mm to (135.6, 106.0), turned to 90 degrees
- moved C4 18.7 mm to (162.5, 100.1)
- moved C3 18.3 mm to (152.1, 101.1), turned to 180 degrees
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Routing:
- net Net-(C2-Pad2): track 0.00 -> 37.8 mm
- net Net-(U5-1IN-): track 0.00 -> 29.1 mm
- net +3.3V: track 0.00 -> 26.9 mm, vias 0 -> 2
- net 2OUT: track 0.00 -> 26.0 mm
- net Net-(U5-1OUT): track 0.00 -> 25.0 mm
- net 2IN+: track 0.00 -> 22.2 mm
- net 1IN+: track 0.00 -> 19.2 mm
- net 2IN-: track 0.00 -> 15.8 mm, vias 0 -> 2
- net Net-(C5-Pad1): track 0.00 -> 6.79 mm
- net +5V: track 0.00 -> 4.97 mm
- net GND: track 0.00 -> 4.37 mm
- net Net-(C3-Pad1): track 0.00 -> 3.62 mm

Commit message: PCB V2
Parts:
- moved C5 11.2 mm to (155.5, 105.0)
- moved C1 7.18 mm to (136.5, 109.0), turned to 180 degrees
- moved R4 6.71 mm to (144.5, 95.0)
- moved C2 6.41 mm to (140.0, 99.0)
- moved R6 5.65 mm to (162.0, 99.0), turned to -90 degrees
- moved R2 4.99 mm to (136.5, 106.0)
- moved C7 4.92 mm to (134.6, 94.5), turned to 0 degrees
- moved R7 4.87 mm to (155.0, 99.0), turned to -90 degrees
- moved R3 4.52 mm to (140.0, 105.0)
- moved C4 4.11 mm to (158.5, 99.0), turned to -90 degrees
- moved C3 4.06 mm to (149.5, 98.0)
- moved R5 3.30 mm to (155.5, 112.0), turned to -90 degrees
- moved R1 2.47 mm to (136.5, 112.0), turned to 180 degrees
Routing:
- net +5V: track 4.97 -> 45.9 mm
- net Net-(U5-1IN-): track 29.1 -> 18.2 mm
- net Net-(U5-1OUT): track 25.0 -> 16.0 mm
- net 1IN+: track 19.2 -> 11.4 mm
- net 2IN+: track 22.2 -> 15.7 mm
- net Net-(C2-Pad2): track 37.8 -> 32.6 mm
- net GND: track 4.37 -> 0.00 mm
- net 2IN-: track 15.8 -> 12.8 mm
- net Net-(C5-Pad1): track 6.79 -> 4.29 mm
