File: KiCAD/Radar.kicad_pcb (KiCad board)
At the start: 2 copper layers, 18 parts, among them U3 HB100, U4 NUCLEO-L432KC, U5 LM358DR

Commit message: PCB V5
Parts:
- moved R4 15.0 mm to (159.5, 95.0)
- moved C7 8.70 mm to (136.5, 103.0)
- moved U4 5.35 mm to (147.2, 124.9)
- moved R6 2.55 mm to (159.5, 99.5)
- moved C4 2.04 mm to (156.5, 99.4)
- moved C3 1.56 mm to (148.0, 98.4)
- moved R7 1.56 mm to (153.5, 99.4)
Routing:
- net +5V: track 45.9 -> 34.3 mm
- net 2OUT: track 26.0 -> 18.4 mm
- net +3.3V: track 27.2 -> 20.5 mm
- net Net-(U5-1IN-): track 18.2 -> 15.5 mm
- net Net-(U5-1OUT): track 16.0 -> 14.3 mm
- net Net-(C2-Pad2): track 32.6 -> 31.3 mm

Commit message: PCB final version
Parts:
- added REF**: MountingHole_2.7mm_M2.5, MountingHole:MountingHole_2.7mm_M2.5, F.Cu at (122.0, 45.0)
- added REF**: MountingHole_2.7mm_M2.5, MountingHole:MountingHole_2.7mm_M2.5, F.Cu at (180.0, 45.0)
- added REF**: MountingHole_2.7mm_M2.5, MountingHole:MountingHole_2.7mm_M2.5, F.Cu at (122.0, 140.0)
- added REF**: ESD-Logo_6.6x6mm_SilkScreen, Symbol:ESD-Logo_6.6x6mm_SilkScreen, F.Cu at (179.5, 101.8)
- added REF**: MountingHole_2.7mm_M2.5, MountingHole:MountingHole_2.7mm_M2.5, F.Cu at (180.0, 140.0)
- moved C7 2.00 mm to (134.5, 103.0)
Routing:
- net GND: track 0.00 -> 94.0 mm, vias 0 -> 42
- net Net-(C2-Pad2): track 31.3 -> 36.0 mm, vias 0 -> 1
- net +5V: track 34.3 -> 35.3 mm
- added copper zone on B.Cu, net GND
- added copper zone on F.Cu, net GND
Other:
- board outline added: 69 x 107 mm
- board text added: "Mateusz Witczak"
